File: A203-V2-Expansion-Board.brd (EAGLE design)
At the start: 87 x 65 mm, 67 parts, among them IC1 FE1.1S, IC2 SN74HC595DR, M1 ICM-42688-P-MODULE-PINHEADER, M2 USB-TO-QUAD-RS-485-CONV-MODUL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

Commit message: Create Rev. 2
Parts:
- added JP10, JP11, JP14, JP15, JP16, JP17: SHORTLAND, Shortland:SHORTLAND
- added SW1: SKRPACE010, SKRPACE010:SKRPACE010
- moved JP3 11.6 mm to (15.6, 12.7), turned to 0 degrees
- moved JP5 11.5 mm to (17.5, 10.2)
- moved JP9 10.5 mm to (15.6, 5.08), turned to 270 degrees
- moved JP6 9.16 mm to (15.6, 10.2), turned to 0 degrees
- moved JP7 4.85 mm to (22.9, 5.08), turned to 180 degrees
- moved JP1 4.07 mm to (22.9, 12.7)
- moved JP4 4.07 mm to (22.9, 10.2), turned to 180 degrees
- moved JP2 3.38 mm to (17.5, 12.7), turned to 180 degrees
- moved JP8 2.22 mm to (17.5, 5.08), turned to 270 degrees
Connections:
- new net CORE_BOARD_SCL: CH2.4, JP16.1, JP17.1
- new net CORE_BOARD_SDA: CH2.3, JP14.1, JP15.1
- net +3V3: now also JP10.2; no longer JP6.2
- net AP_CS: now also JP10.1, JP11.1; no longer JP8.1, JP9.1
- net AP_SCL/SCLK: now also JP3.1
- net AP_SDA/SDI: now also JP5.1, JP6.1; no longer JP3.1
- net AP_SDO/ADO: now also JP8.1, JP9.1; no longer JP5.1, JP6.1
- net GND: now also JP9.2, SW1.3, SW1.4; no longer JP7.2
- net I2C1_SCL: now also JP17.2, JP3.2; no longer CH2.4, JP2.2
- net I2C1_SDA: now also JP15.2, JP6.2; no longer CH2.3, JP4.2
- net ID_I2C_SCL: now also JP16.2, JP2.2
- net ID_I2C_SDA: now also JP14.2, JP5.2
- net RECOVERY: now also SW1.1, SW1.2
- net SPI0_CS0: now also JP11.2; no longer JP9.2
- net SPI0_MISO: now also JP7.2; no longer JP5.2
- net SPI0_MOSI: now also JP4.2; no longer JP3.2
Routing:
- net CORE_BOARD_SCL: track 0.00 -> 68.3 mm
- net CORE_BOARD_SDA: track 0.00 -> 46.0 mm
- net ID_I2C_SDA: track 0.00 -> 36.6 mm, vias 0 -> 1
- net USBDN-DM2: track 99.0 -> 66.6 mm, vias 0 -> 4
- net AP_SDO/ADO: track 72.3 -> 103.6 mm, vias 0 -> 3
- net USBDN-DM3: track 112.2 -> 81.6 mm
- net I2C1_SDA: track 46.5 -> 74.1 mm, vias 3 -> 1
- net ID_I2C_SCL: track 0.00 -> 22.6 mm
- net RECOVERY: track 0.00 -> 18.9 mm
- net D-RX: track 40.0 -> 21.2 mm, vias 2 -> 0
- net SPI0_CS0: track 36.8 -> 20.0 mm, vias 3 -> 1
- net B-RX: track 46.3 -> 33.1 mm, vias 2 -> 4
- net USBDN-DP2: track 78.6 -> 66.6 mm, vias 2 -> 6
- net B-DM: track 50.9 -> 39.0 mm, vias 0 -> 1
- net +3V3: track 149.5 -> 137.8 mm
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Other:
- board text added: "A203 V2 Expansion Board Rev. 2 Designed by Masato Kubotera on June 19, 2023."
- board text added: "Bus 1"
- board text added: "Bus 8"
- board text added: "Recovery"
- board text added: "Select Core Board's I2C Bus"
- board text removed: "A203 V2 Expansion Board Rev. 1 Designed by Masato Kubotera on May 31, 2023."
