File: A203-V2-Expansion-Board.sch (EAGLE design)
At the start: 67 parts, among them IC1 FE1.1S, IC2 SN74HC595DR, M1 ICM-42688-P-MODULE-PINHEADER, M2 USB-TO-QUAD-RS-485-CONV-MODUL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

Commit message: Fixed wiring error on USB DN Port 3
Connections:
- removed net USB-DN-DM3: M2.USB-DM
- removed net USB-DN-DP3: M2.USB-DP
- net USBDN-DM3: now also M2.USB-DM
- net USBDN-DP3: now also M2.USB-DP
Other:
- note added: "May 31, 2023"
- note removed: "May 22, 2023"
Changed lines of the file:
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@@
 <text x="391.16" y="15.24" size="5.08" layer="94" ratio="10" align="center-left">1</text>
 <text x="396.24" y="5.08" size="5.08" layer="94" ratio="10" align="center-left">1/1</text>
-<text x="307.34" y="5.08" size="5.08" layer="94" ratio="10" align="center-left">May 22, 2023</text>
+<text x="307.34" y="5.08" size="5.08" layer="94" ratio="10" align="center-left">May 31, 2023</text>
 <text x="307.34" y="25.4" size="5.08" layer="94" ratio="10" align="center-left">A203 V2 Expansion Board</text>
 <text x="287.02" y="167.64" size="1.778" layer="97" ratio="10" rot="R90" align="center">Hub Active/Suspend Indicator</text>
@@
 <label x="241.3" y="226.06" size="1.778" layer="95" rot="R180"/>
 <pinref part="IC1" gate="G$1" pin="DP1"/>
-</segment>
-</net>
-<net name="USB-DN-DP3" class="0">
-<segment>
-<wire x1="335.28" y1="99.06" x2="330.2" y2="99.06" width="0.1524" layer="91"/>
-<label x="330.2" y="99.06" size="1.778" layer="95" rot="R180"/>
-<pinref part="M2" gate="G$1" pin="USB-DP"/>
-</segment>
-</net>
-<net name="USB-DN-DM3" class="0">
-<segment>
-<wire x1="335.28" y1="101.6" x2="330.2" y2="101.6" width="0.1524" layer="91"/>
-<label x="330.2" y="101.6" size="1.778" layer="95" rot="R180"/>
-<pinref part="M2" gate="G$1" pin="USB-DM"/>
 </segment>
 </net>
@@
 <pinref part="IC1" gate="G$1" pin="DP3"/>
 </segment>
+<segment>
+<wire x1="335.28" y1="99.06" x2="330.2" y2="99.06" width="0.1524" layer="91"/>
+<label x="330.2" y="99.06" size="1.778" layer="95" rot="R180"/>
+<pinref part="M2" gate="G$1" pin="USB-DP"/>
+</segment>
 </net>
 <net name="USBDN-DM3" class="0">
@@
 <pinref part="IC1" gate="G$1" pin="DM3"/>
 </segment>
-</net>
+<segment>
+<wire x1="335.28" y1="101.6" x2="330.2" y2="101.6" width="0.1524" layer="91"/>
+<label x="330.2" y="101.6" size="1.778" layer="95" rot="R180"/>
+<pinref part="M2" gate="G$1" pin="USB-DM"/>
+</segment>
+</net>

Commit message: Create Rev. 2
Parts:
- added JP10, JP11, JP14, JP15, JP16, JP17: SHORTLAND, Shortland:SHORTLAND
- added SW1: SKRPACE010, SKRPACE010:SKRPACE010
Connections:
- new net CORE_BOARD_SCL: CH2.4, JP16.1, JP17.1
- new net CORE_BOARD_SDA: CH2.3, JP14.1, JP15.1
- net +3V3: now also JP10.2; no longer JP6.2
- net AP_CS: now also JP10.1, JP11.1; no longer JP8.1, JP9.1
- net AP_SCL/SCLK: now also JP3.1
- net AP_SDA/SDI: now also JP5.1, JP6.1; no longer JP3.1
- net AP_SDO/ADO: now also JP8.1, JP9.1; no longer JP5.1, JP6.1
- net GND: now also JP9.2, SW1.2; no longer JP7.2
- net I2C1_SCL: now also JP17.2, JP3.2; no longer CH2.4, JP2.2
- net I2C1_SDA: now also JP15.2, JP6.2; no longer CH2.3, JP4.2
- net ID_I2C_SCL: now also JP16.2, JP2.2
- net ID_I2C_SDA: now also JP14.2, JP5.2
- net RECOVERY: now also SW1.1
- net SPI0_CS0: now also JP11.2; no longer JP9.2
- net SPI0_MISO: now also JP7.2; no longer JP5.2
- net SPI0_MOSI: now also JP4.2; no longer JP3.2
Other:
- note added: "2"
- note added: "June 19, 2023"
- note added: "Recovery Switch"
- note removed: "1"
- note removed: "May 31, 2023"
- moved on the sheet: CH2, IC2, JP1, JP2, JP3, JP4, JP5, JP6, JP7, JP8, JP9, LED10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
